File: wakaba/wakaba.kicad_sch (KiCad schematic)
At the start: 134 parts, among them J1 USB_C_Receptacle_USB2.0, J10 M1, J11 M2, J2 Conn_01x06_Socket, J3 Battery, J4 Attiny_program, J5 Conn_01x04_Pin, J6 Conn_01x04_Pin, J7 Conn_01x06_Socket, J8 Conn_01x06_Socket, J9 Conn_01x06_Socket, Q1 MTP4835i3, Q2 IRFML8244, Q3 IRFML8244, SW1 SW_MEC_5E, SW2 SW_SPDT, SW3 SW_SPDT, SW4 SW_DIP_x04, U10 NSI45090, U11 AD8604, U12 MA702, U13 MA702, U14 BNO055, U15 DRV8836DSSR, U2 MIC5219-5.0YM5, U3 INA219AxDCN, U4 ATtiny85-20S, U5 TLP290, U6 ACS712LLCTR-10AB-T, U7 NCP1117-ADJ_SOT223, U8 MIC5219-3.3YM5, U9 NSI45090, Y1 12.000MHz, Y2 32.768kHz

Commit message: 3v3に統一作業WIP
Parts:
- removed C10: 2.2u, symbol Device:C
- removed C19: 22u, symbol Device:C
- removed C20: C, symbol Device:C
- removed C9: 470p, symbol Device:C
- removed D1: 1N4007, symbol Device:D
- removed RV1: 5k, symbol Device:R_Potentiometer
- removed SW3: SW_SPDT, symbol Switch:SW_SPDT
- removed U2: MIC5219-5.0YM5, Package_TO_SOT_SMD:SOT-23-5, symbol Regulator_Linear:MIC5219-3.3YM5
- removed U7: NCP1117-ADJ_SOT223, Package_TO_SOT_SMD:SOT-223-3_TabPin2, symbol Regulator_Linear:NCP1117-ADJ_SOT223
- added D1: 1N4148W, Diode_SMD:D_SOD-123, symbol Diode:1N4148W
- added D18, D19: SS2040, symbol Device:D_Schottky
- added Q4, Q5: AO3401A, Package_TO_SOT_SMD:SOT-23, symbol Transistor_FET:AO3401A
- added R44: R, symbol Device:R
- added SW5: SW_SPST, symbol Switch:SW_SPST
- R11: value 1k -> 10k
Connections:
- net +3V3: now also C15.1, C18.1, U3.4 (VS), U6.8 (VCC)
- net GND: now also R44.2, SW5.1 (A)
- net SUB5V: now also D11.2 (A), D19.1 (K); no longer C15.1, C18.1, J4.1 (Pin_1), U3.4 (VS), U6.8 (VCC)
- net VBAT: now also R11.1, Q5.2 (S); no longer Q1.3 (S), R8.2, R9.1, U3.1 (IN+)
- net VCC: now also U8.1 (IN), U8.3 (EN)
- net DCDC_CE: now reaches R11.2
- net DCDC_CE: now also SW5.2 (B)
- net at J1.A4 (VBUS), J1.A9 (VBUS), J1.B4 (VBUS)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: now also J5.1 (Pin_1)
- removed net +5V: D11.2 (A), U8.1 (IN), U8.3 (EN)
- net BAT_CHG renamed VBUS
- net VBUS: now also D1.2 (A), D18.2 (A)
- new net: D1.1 (K), Q4.1 (G), Q5.1 (G), R44.1
- new net: D19.2 (A), J4.1 (Pin_1)
- new net: Q4.3 (D), Q5.3 (D)
- new net VDD: D18.1 (K), Q1.3 (S), Q4.2 (S), R8.2, R9.1, U3.1 (IN+)
- no-connect marks 42 -> 41
Other:
- note removed: "Considering"
- note removed: "Main 5V regulator"

Commit message: wip
Parts:
- removed R11: 10k, symbol Device:R
- removed SW5: SW_SPST, symbol Switch:SW_SPST
- added C10: 2.2u, symbol Device:C
- added C9: 470p, symbol Device:C
- added F1: 0ZCH0075AF2E, Resistor_SMD:R_1210_3225Metric_Pad1.30x2.65mm_HandSolder, symbol Device:Polyfuse
- added SW3: SW_Push, symbol Switch:SW_Push
- added U2: MIC5219-3.3YM5, Package_TO_SOT_SMD:SOT-23-5, symbol Regulator_Linear:MIC5219-3.3YM5
Connections:
- net +3V3: no longer C15.1, C18.1, U3.4 (VS), U6.8 (VCC)
- net GND: now also C10.2, C9.2, SW3.2, U2.2 (GND); no longer R40.2, U1.24 (P204)
- net SUB5V: no longer C16.1, R41.1, R42.1, U4.8 (VCC)
- net VDD: now also F1.2, U2.1 (IN), U2.3 (EN); no longer D18.1 (K), Q4.2 (S)
- net BUZZ: now reaches U1.30 (P302)
- new net: D18.1 (K), F1.1, Q4.2 (S)
- new net: C9.1, U2.4 (BP)
- new net SUB3V3: C10.1, C15.1, C16.1, C18.1, R41.1, R42.1, U2.5 (OUT), U3.4 (VS), U4.8 (VCC), U6.8 (VCC)
- new net USER_PUSHSW: R40.2, SW3.1, U1.24 (P204)
- no-connect marks 41 -> 40
Other:
- moved on the sheet: C15, D1, D18, Q4, Q5, R34, R35, R41, R42, R43, R44, R6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

Commit message: kossanレビュー後修正WIP
Parts:
- C12, C13: value 1n -> 1u
Connections:
- net ENC_CS_R: now also U1.38 (P113); no longer U1.37 (P112)
Changed lines of the file:
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@@
   (no_connect (at 100.33 121.92))
   (no_connect (at 270.51 191.77))
+  (no_connect (at 100.33 144.78))
   (no_connect (at 270.51 189.23))
   (no_connect (at 100.33 185.42))
-  (no_connect (at 100.33 147.32))
   (no_connect (at 270.51 196.85))
   (no_connect (at 100.33 132.08))
@@
     )
   )
-  (global_label "ENC_CS_R" (shape input) (at 100.33 144.78 180) (fields_autoplaced)
-    (effects (font (size 1.27 1.27)) (justify right))
-    (property "Intersheetrefs" "${INTERSHEET_REFS}" (at 87.9106 144.78 0)
+  (global_label "ENC_CS_R" (shape input) (at 100.33 147.32 180) (fields_autoplaced)
+    (effects (font (size 1.27 1.27)) (justify right))
+    (property "Intersheetrefs" "${INTERSHEET_REFS}" (at 87.9106 147.32 0)
       (effects (font (size 1.27 1.27)) (justify right) hide)
     )
@@
       (effects (font (size 1.27 1.27)) (justify left))
     )
-    (property "Value" "1n" (at 278.13 195.58 0)
+    (property "Value" "1u" (at 278.13 195.58 0)
       (effects (font (size 1.27 1.27)) (justify left))
     )
@@
       (effects (font (size 1.27 1.27)) (justify left))
     )
-    (property "Value" "1n" (at 278.13 146.05 0)
-      (effects (font (size 1.27 1.27)) (justify left))
-    )
+    (property "Value" "1u" (at 278.13 146.05 0)
+      (effects (font (size 1.27 1.27)) (justify left))
+    )

Commit message: 保護回路削除
Parts:
- removed C10: 2.2u, symbol Device:C
- removed C15, C16, C18: 0.1u, symbol Device:C
- removed C17: 1n, symbol Device:C
- removed C9: 470p, symbol Device:C
- removed D11, D13: LED, symbol Device:LED
- removed D19: SS2040, symbol Device:D_Schottky
- removed J3: Battery, symbol Connector:Conn_01x02_Pin
- removed J4: Attiny_program, symbol Connector:Conn_01x06_Pin
- removed Q1: MTP4835i3, symbol Device:Q_PMOS_GDS
- removed R10: 301, symbol Device:R
- removed R37, R39: R, symbol Device:R
- removed R41, R42, R43, R6, R7, R9: 10k, symbol Device:R
- removed R8: 100, symbol Device:R
- removed U2: MIC5219-3.3YM5, Package_TO_SOT_SMD:SOT-23-5, symbol Regulator_Linear:MIC5219-3.3YM5
- removed U3: INA219AxDCN, Package_TO_SOT_SMD:SOT-23-8_Handsoldering, symbol Sensor_Energy:INA219AxDCN
- removed U4: ATtiny85-20S, Package_SO:SOIC-8W_5.3x5.3mm_P1.27mm, symbol MCU_Microchip_ATtiny:ATtiny85-20S
- removed U5: TLP290, Package_SO:SOP-4_4.4x2.6mm_P1.27mm, symbol Isolator:TLP290
- removed U6: ACS712LLCTR-10AB-T, Package_SO:SOIC-8_3.9x4.9mm_P1.27mm, symbol Sensor_Current:ACS712xLCTR-30A
- R36: value R -> 50
- R38: value R -> 20
- RN1: value 1k -> 20
Connections:
- net VDD is gone; now on net VCC: F1.2
Other:
- note removed: "Battery Protection"

Commit message: パターン一旦完成
Parts:
- removed C11, C7: 10p, symbol Device:C
- removed J2, J7: Conn_01x06_Socket, symbol Connector:Conn_01x06_Socket
- removed R12, R17: 100, symbol Device:R
- removed RN1: 20, Resistor_THT:R_Array_SIP5, symbol Device:R_Pack04_SIP_Split
- removed SW2: SW_SPDT, symbol Switch:SW_SPDT
- removed U10, U9: NSI45090, Package_TO_SOT_SMD:TO-252-3_TabPin2, symbol Regulator_Linear:LM1117DT-ADJ
- removed Y1: 12.000MHz, symbol Device:Crystal
- added J12, J2, J4, J7: Conn_01x03_Pin, wakaba:vertical_pcb_conn, symbol Connector:Conn_01x03_Pin
- added J3: 5055680271, CON_5055680271, symbol 2023-11-13_14-47-42:5055680271
- added R6, R7, R8, R9: 20, Resistor_SMD:R_0603_1608Metric_Pad0.98x0.95mm_HandSolder, symbol Device:R
- added SW2: SW_Push_SPDT, wakaba:SSAJ120, symbol Switch:SW_Push_SPDT
- added Y1: CSTNE12M0G520000R0, Crystal:Resonator_SMD_Murata_CSTxExxV-3Pin_3.0x1.1mm, symbol Device:Resonator_Small
- C1, C12, C13, C14, C2, C21, C22, C23, C24, C25, C26, C27, C28, C29, C30, C31, C32, C33, C34, C35, C4, C5, C6: footprint (none) -> Capacitor_SMD:C_0603_1608Metric_Pad1.08x0.95mm_HandSolder
- C3, C8: footprint (none) -> Capacitor_SMD:C_0805_2012Metric_Pad1.18x1.45mm_HandSolder
- D10, D12, D14, D15, D16, D17: footprint (none) -> LED_SMD:LED_0603_1608Metric_Pad1.05x0.95mm_HandSolder
- D18: footprint (none) -> Diode_SMD:D_SOD-123F
- D2, D3, D4, D5, D6, D7, D8, D9: footprint (none) -> LED_THT:LED_D5.0mm_Horizontal_O1.27mm_Z3.0mm
- J1: footprint (none) -> Connector_USB:USB_C_Receptacle_G-Switch_GT-USB-7010ASV
- J10, J11: footprint (none) -> Connector_PinHeader_1.27mm:PinHeader_1x02_P1.27mm_Vertical
- J5: footprint (none) -> wakaba:pogo_usb
- J6: footprint (none) -> wakaba:pogopad_usb
- J8, J9: footprint (none) -> wakaba:vertical_pcb_conn_base
- JP1: footprint (none) -> Jumper:SolderJumper-2_P1.3mm_Open_RoundedPad1.0x1.5mm
- R1, R13, R14, R15, R16, R18, R19, R2, R20, R21, R22, R23, R24, R25, R26, R27, R28, R29, R3, R30, R31, R32, R33, R34, R35, R36, R38, R4, R40, R5: footprint (none) -> Resistor_SMD:R_0603_1608Metric_Pad0.98x0.95mm_HandSolder
- R44: value R -> 10k; footprint (none) -> Resistor_SMD:R_0603_1608Metric_Pad0.98x0.95mm_HandSolder
- RN2: footprint Resistor_THT:R_Array_SIP8 -> Resistor_SMD:R_Array_Concave_4x0402
- SW1, SW3: footprint (none) -> Button_Switch_SMD:SW_SPST_PTS810
- SW4: footprint (none) -> Button_Switch_SMD:SW_DIP_SPSTx04_Slide_Copal_CHS-04B_W7.62mm_P1.27mm
- U1: value ~ -> R7FA4M1AB3CNB#AC0; footprint Package_QFP:LQFP-64_10x10mm_P0.5mm -> Package_DFN_QFN:QFN-64-1EP_8x8mm_P0.4mm_EP6.5x6.5mm
- U15: footprint DRV8836DSSR:SON50P200X300X80-13N -> wakaba:SON50P200X300X80-13N
- Y2: footprint (none) -> Crystal:Crystal_SMD_2012-2Pin_2.0x1.2mm_HandSoldering
Connections:
- net +3V3: now also J2.1 (Pin_1), J7.1 (Pin_1)
- net GND: now also J12.2 (Pin_2), J3.2, J3.3, J3.4, J4.2 (Pin_2), R6.2, R7.2, R8.2, R9.2, Y1.2
- net VBAT: now also J3.1
- net VCC: now also D5.2 (A); no longer D2.2 (A)
- net at U13.12 (SCLK): now also J12.3 (Pin_3)
- net at U13.4 (MOSI): now also J7.2 (Pin_2)
- net at U13.5 (~{CS}): now also J7.3 (Pin_3)
- net at U13.7 (MISO): now also J12.1 (Pin_1)
- net at Q2.1 (D): now also D3.1 (K)
- net at D16.1 (K): now also R8.1
- net at U1.10 (P212/EXTAL): now also Y1.3
- net at D2.1 (K): now also Q3.1 (D); no longer D3.2 (A)
- net at U1.9 (P213/XTAL): now also Y1.1
- net at R26.1: now also SW2.1 (A)
- net at U1.26 (P201/MD): now also SW2.2 (B)
- net at R3.2: now also SW2.3 (C)
- net at D4.1 (K): now also D2.2 (A); no longer D5.2 (A)
- net at U12.12 (SCLK): now also J4.3 (Pin_3)
- net at U12.4 (MOSI): now also J2.2 (Pin_2)
- net at U12.5 (~{CS}): now also J2.3 (Pin_3)
- net at U12.7 (MISO): now also J4.1 (Pin_1)
- net at D15.1 (K): now also R7.1
- net at D17.1 (K): now also R9.1
- net at D14.1 (K): now also R6.1
- net at D5.1 (K): now also D3.2 (A)
- net BUZZ: no longer names the net of U1.30 (P302)
- no-connect marks 40 -> 41
Other:
- moved on the sheet: D2, D5
